Commit message: 更换台面颜色，更换相机模型

File: config/gazebo_ur10e_with_robotiq_2f_85_camera.urdf (robot description, URDF)
Before this commit: robot ur10e_with_robotiq_2f_85, 25 links, 24 joints
Links:
- link camera_link: geometry collision mesh filename=package://scanner/meshes/collision/scanner.stl; visual mesh filename=package://scanner/meshes/visual/scanner.dae
- link table_base_link: geometry collision mesh filename=package://table/meshes/table_base_link.STL; visual mesh filename=package://table/meshes/table_base_link.dae
