Commit message: 更换moveit规划末端

File: config/gazebo_ur10e_with_robotiq_2f_85.urdf (robot description, URDF)
Before this commit: robot ur10e_with_robotiq_2f_85, 21 links, 20 joints
Links:
- added link finger_center
Joints:
- added joint finger_center_joint: type fixed, parent tool0, child finger_center, origin xyz=0 0 0.16 rpy=0 0 0

File: config/gazebo_ur10e_with_robotiq_2f_85_camera.urdf (robot description, URDF)
Before this commit: robot ur10e_with_robotiq_2f_85, 25 links, 24 joints
Links:
- added link finger_center
Joints:
- added joint finger_center_joint: type fixed, parent tool0, child finger_center, origin xyz=0 0 0.16 rpy=0 0 0

File: config/gazebo_ur10e_with_robotiq_2f_85_camera_couple.urdf (robot description, URDF)
Before this commit: robot ur10e_with_robotiq_2f_85, 26 links, 25 joints
Links:
- added link finger_center
Joints:
- added joint finger_center_joint: type fixed, parent tool0, child finger_center, origin xyz=0 0 0.16 rpy=0 0 0

File: config/gazebo_ur10e_with_robotiq_2f_85_camera（复件）.urdf (robot description, URDF)
Before this commit: robot ur10e_with_robotiq_2f_85, 25 links, 24 joints
Links:
- added link finger_center
Joints:
- added joint finger_center_joint: type fixed, parent tool0, child finger_center, origin xyz=0 0 0.16 rpy=0 0 0

File: config/gazebo_ur10e_with_robotiq_2f_85_eyeinhand.urdf (robot description, URDF)
Before this commit: robot ur10e_with_robotiq_2f_85, 26 links, 25 joints
Links:
- removed link table_base_link
- removed link table_link
- link camera_link: mass 0.1 -> None; geometry visual cylinder length=0.01 radius=0.01
Joints:
- removed joint table_base_joint
- removed joint table_base_table_joint
- joint camera_joint: origin xyz=0.3 -0.8 1.0 rpy=0 1.5708 0 -> xyz=0 0.0 0.15 rpy=0 -1.5708 0; parent base_link -> wrist_3_link
- joint robotiq_85_base_joint: origin xyz=0 0 0.004 rpy=0 -1.5707963267948966 3.141592653589793 -> xyz=0 0 0.007 rpy=0 -1.5707963267948966 3.141592653589793
- joint world_table_base_joint: child table_base_link -> base_link
